Commit message: camera - need to modify

File: catkin_ws/src/my_mobile/urdf/mobile_robot.xacro (robot description, xacro)
@@ -49,4 +49,5 @@
     </visual>
   </link>
+  <!--
 	<link name="sensor_laser">
 		<inertial>
@@ -74,4 +75,32 @@
 		<child link="sensor_laser"/>
 	</joint>
+	-->
+	<!-- Camera -->
+	<link name="link_camera">
+		<inertial>
+			<origin xyz="0 0 0" rpy="0 0 0"/>
+			<mass value="1"/>
+			<inertia ixx="1e-6" ixy="0" ixz="0" iyy="1e-6" iyz="0" izz="1e-6"/>
+		</inertial>
+		<visual>
+			<origin xyz="0 0 0" rpy="0 0 0"/>
+			<geometry>
+			<box size="0.05 0.05 0.05"/>
+			</geometry>
+			<material name="orange"/>
+		</visual>
+		<collision>
+			<origin xyz="0 0 0" rpy="0 0 0"/>
+			<geometry>
+			<box size="0.05 0.05 0.05"/>
+			</geometry>
+		</collision>
+	</link>
+	<joint name="joint_camera" type="fixed">
+		<!-- <axis xyz="0 0 1"/> -->
+		<origin xyz="0 0 0.15" rpy="0 0 0"/>
+		<parent link="link_chassis"/>
+		<child link="link_camera"/>
+	</joint>
   <xacro:link_wheel name="link_right_wheel" />
   <xacro:joint_wheel name="joint_right_wheel" child="link_right_wheel" origin_xyz="-0.05 0.15 0" />
