Commit message: mobile robot with laser sensor and camera

File: catkin_ws/src/my_mobile/urdf/macros.xacro (robot description, xacro)
@@ -32,8 +32,7 @@
       </joint>
     </xacro:macro>
-	<xacro:macro name="cylinder_inertia" params="mass r l">
-		<inertia ixx="${mass*(3*r*r+l*l)/12}" ixy="0" ixz="0"
-				iyy="${mass*(3*r*r+l*l)/12}" iyz="0"
-				izz="${mass*(r*r)/2}"/>
-	</xacro:macro>
+    <xacro:macro name="cylinder_inertia" params="mass r l">
+        <inertia ixx="${mass*(3*r*r+l*l)/12}" ixy ="0" ixz ="0"
+		iyy="${mass*(3*r*r+l*l)/12}" iyz ="0" izz="${mass*(r*r)/2}"/>
+    </xacro:macro>
 </robot>

File: catkin_ws/src/my_mobile/urdf/mobile_robot.xacro (robot description, xacro)
@@ -49,58 +49,56 @@
     </visual>
   </link>
-  <!--
-	<link name="sensor_laser">
-		<inertial>
-			<origin xyz="0 0 0" rpy="0 0 0"/>
-			<mass value="1"/>
-			<xacro:cylinder_inertia mass="1" r="0.05" l="0.1"/>
-		</inertial>
-		<visual>
-			<origin xyz="0 0 0" rpy="0 0 0"/>
-			<geometry>
-			<cylinder radius="0.05" length="0.1"/>
-			</geometry>
-			<material name="white"/>
-		</visual>
-		<collision>
-			<origin xyz="0 0 0" rpy="0 0 0"/>
-			<geometry>
-			<cylinder radius="0.05" length="0.1"/>
-			</geometry>
-		</collision>
-	</link>
-	<joint name="joint_sensor_laser" type="fixed">
-		<origin xyz="0.15 0 0.05" rpy="0 0 0"/>
-		<parent link="link_chassis"/>
-		<child link="sensor_laser"/>
-	</joint>
-	-->
-	<!-- Camera -->
-	<link name="link_camera">
-		<inertial>
-			<origin xyz="0 0 0" rpy="0 0 0"/>
-			<mass value="1"/>
-			<inertia ixx="1e-6" ixy="0" ixz="0" iyy="1e-6" iyz="0" izz="1e-6"/>
-		</inertial>
-		<visual>
-			<origin xyz="0 0 0" rpy="0 0 0"/>
-			<geometry>
-			<box size="0.05 0.05 0.05"/>
-			</geometry>
-			<material name="orange"/>
-		</visual>
-		<collision>
-			<origin xyz="0 0 0" rpy="0 0 0"/>
-			<geometry>
-			<box size="0.05 0.05 0.05"/>
-			</geometry>
-		</collision>
-	</link>
-	<joint name="joint_camera" type="fixed">
-		<!-- <axis xyz="0 0 1"/> -->
-		<origin xyz="0 0 0.15" rpy="0 0 0"/>
-		<parent link="link_chassis"/>
-		<child link="link_camera"/>
-	</joint>
+  <link name="sensor_laser">
+    <inertial>
+        <origin xyz="0 0 0" rpy="0 0 0"/>
+	<mass value="1"/>
+	<xacro:cylinder_inertia mass="1" r="0.05" l="0.1"/>
+    </inertial>
+    <visual>
+	<origin xyz="0 0 0" rpy="0 0 0"/>
+	<geometry>
+	<cylinder radius="0.05" length="0.1"/>
+        </geometry>
+	<material name="white"/>
+    </visual>
+    <collision>
+	<origin xyz="0 0 0" rpy="0 0 0"/>
+	<geometry>
+	<cylinder radius="0.05" length="0.1"/>
+        </geometry>
+    </collision>
+  </link>
+  <joint name="joint_sensor_laser" type="fixed">
+    <origin xyz="0.15 0 0.05" rpy="0 0 0"/>
+    <parent link="link_chassis"/>
+    <child link="sensor_laser"/>
+  </joint>
+  <!-- Camera -->
+  <link name="link_camera">
+    <inertial>
+      <origin xyz="0 0 0" rpy="0 0 0"/>
+      <mass value="1"/>
+      <inertia ixx="1e-6" ixy="0" ixz="0" iyy="1e-6" iyz="0" izz="1e-6"/>
+    </inertial>
+    <visual>
+      <origin xyz="0 0 0" rpy="0 0 0"/>
+      <geometry>
+      <box size="0.05 0.05 0.05"/>
+      </geometry>
+      <material name="orange"/>
+    </visual>
+    <collision>
+      <origin xyz="0 0 0" rpy="0 0 0"/>
+      <geometry>
+      <box size="0.05 0.05 0.05"/>
+      </geometry>
+    </collision>
+  </link>
+  <joint name="joint_camera" type="fixed">
+    <!-- <axis xyz="0 0 1"/> -->
+    <origin xyz="0 0 0.05" rpy="0 0 0"/>
+    <parent link="sensor_laser"/>
+    <child link="link_camera"/>
+  </joint>
   <xacro:link_wheel name="link_right_wheel" />
   <xacro:joint_wheel name="joint_right_wheel" child="link_right_wheel" origin_xyz="-0.05 0.15 0" />
